File: SVF/2164_svf_single_plane_smd.sch (EAGLE design)
At the start: 88 parts, among them IC1 SSM2164S, IC2 TL072, IC3 TL072, IC4 TL072, IC5 TL072, IC6 TL072, U1 THONKICONNNEW, U2 THONKICONNNEW, U3 THONKICONNNEW, U4 THONKICONNNEW, U5 THONKICONNNEW, U6 THONKICONNNEW

Commit message: Add V1.7 files for SVF
Parts:
- removed D5, D6: 1N5817, diode:SCHOTTKY-DIODEDO35-7
- removed HEADR1, HEADR2, HEADR3, HEADR4: (no value), MusicThingModular:10PIN_BACKSIDE
- added C25, C26: 100n, rcl:C-EUC0603
- added D7: BAT854W, nxp_60:1PS70SB10
- added VD1, VD2: SS12L, diode:DIODE-SCHOTTKY-SMA
- renumbered R30 to R32
Connections:
- removed net BP_CONN: HEADR1.6, U4.TIP
- removed net CUTOFF_POT1: HEADR1.3, VR4.S
- removed net CUTOFF_POT2: HEADR1.5, VR4.A
- removed net CV1_POT: HEADR1.7, VR3.S
- removed net CV2_POT1: HEADR1.2, VR5.E
- removed net CV2_POT2: HEADR1.1, VR5.A
- removed net HP_CONN: HEADR1.10, U6.TIP
- removed net INPUT_POT: HEADR1.9, VR2.S
- removed net LP_CONN: HEADR1.8, U5.TIP
- removed net N$38: D5.C, L1.2
- removed net N$41: D6.A, L2.2
- removed net RESO_POT1: HEADR3.2, VR1.E, VR1.S
- removed net RESO_POT2: HEADR3.1, VR1.A
- removed net TO_BP_CONN: HEADR2.5, R22.2
- removed net TO_CUTOFF_POT1: HEADR2.4, R15.1
- removed net TO_CUTOFF_POT2: HEADR2.6, R29.2
- removed net TO_CV1_POT: HEADR2.8, R14.1
- removed net TO_HP_CONN: HEADR2.9, R26.2
- removed net TO_INPUT_POT: HEADR2.10, R5.1
- removed net TO_LP_CONN: HEADR2.7, R24.2
- new net N$11: R29.2, VR4.A
- new net N$19: R14.1, VR3.S
- new net N$20: R5.1, VR2.S
- new net N$22: R26.2, U6.TIP
- new net N$24: R24.2, U5.TIP
- new net N$25: R22.2, U4.TIP
- new net N$3: R15.1, VR4.S
- new net N$32: L1.2, VD2.C
- new net N$35: L2.2, VD1.A
- net AGND: now also C25.1, C26.2, D7.K; no longer HEADR1.4, HEADR2.3, HEADR3.10, HEADR3.3, HEADR3.4, HEADR3.5, HEADR3.6, HEADR3.7, HEADR3.8, HEADR3.9, HEADR4.10, HEADR4.3, HEADR4.4, HEADR4.5, HEADR4.6, HEADR4.7, HEADR4.8, HEADR4.9
- net N$42: now also VD1.C; no longer D6.C
- net N$43: now also VD2.A; no longer D5.A
- net TO_CV2_POT1: now also VR5.E; no longer HEADR2.1
- net TO_CV2_POT2: now also VR5.A; no longer HEADR2.2
- net TO_RESO_POT1: now also VR1.E, VR1.S; no longer HEADR4.1
- net TO_RESO_POT2: now also VR1.A; no longer HEADR4.2
- net V+: now also C25.2
- net V-: now also C26.1, D7.A
Other:
- moved on the sheet: C19, C20, C21, C22, C23, C24, IC1E, IC2G3, IC3G3, IC4G3, IC5G3, VR4
